Commit message: Final commit

File: gesture_ws/src/niyantrak_description/urdf/diff_drive.xacro (robot description, xacro)
@@ -16,11 +16,4 @@
         <material> Gazebo/Grey </material>
     </gazebo>
-<!--
-    <gazebo reference="right_middle_wheel_link">
-        <material> Gazebo/White </material>
-    </gazebo>
-    <gazebo reference="left_middle_wheel_link">
-        <material> Gazebo/White </material>
-    </gazebo> -->
     <gazebo>
         <plugin name="diff_drive_1" filename="libgazebo_ros_diff_drive.so">

File: gesture_ws/src/niyantrak_description/urdf/lidar.xacro (robot description, xacro)
@@ -27,5 +27,5 @@
         </collision>
         <inertial>
-            <mass value="${m}" /> <!-- Example mass in kg -->
+            <mass value="${m}" />
             <inertia
                 ixx="${(m/12) * (3*r*r + L*L)}"
